File: Hardware/BleSmartLock/BleSmartLock.kicad_sch (KiCad schematic)
At the start: 4 parts

Commit message: Ajout carte BleSmartLock
Other:
- company: (none) -> antoine163
- title: (none) -> Ble Smart Lock
Changed lines of the file:
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@@
 	(generator_version "8.0")
 	(paper "A4")
+	(title_block
+		(title "Ble Smart Lock")
+		(date "2024-03-30")
+		(rev "v1.0")
+		(company "antoine163")
+	)
 	(wire
 		(pts
