File: Hardware/BleSmartLock/BleSmartLock_Bluenrg.kicad_sch (KiCad schematic)
At the start: 21 parts, among them J5 Conn_01x01, J6 Conn_ST_STDC14, J7 Conn_01x06, SW1 SW_Push, U3 BLUENRG-M2SA

Commit message: Ajout carte BleSmartLock
Parts:
- removed J5: Conn_01x01, Connector_PinHeader_2.54mm:PinHeader_1x01_P2.54mm_Vertical, symbol Connector_Generic:Conn_01x01
- added D5: ESD5Z3.3T1G, Diode_SMD:D_SOD-523, symbol Diode:ESD5Zxx
- added SW1: SW_Push, Button_Switch_SMD:SW_SPST_PTS645, symbol Switch:SW_Push
- renumbered D5 to D6, D6 to D7, D7 to D8, D8 to D9, SW1 to SW2
Connections:
- net GND: now also D5.2 (A), SW1.2
- net LIGHT_BLUE: now also U3.18 (DIO1); no longer U3.16 (DIO2)
- net LIGHT_GREEN: now also U3.16 (DIO2); no longer U3.18 (DIO1)
- net LIGHT_PWM: now also U3.3 (DIO4); no longer U3.17 (DIO3)
- net LIGHT_WHITE: now also U3.17 (DIO3); no longer U3.3 (DIO4)
- net M2_~{RESET}: now also D5.1 (K), SW1.1
- net OPENED: now also U3.9 (DIO6); no longer U3.20 (DIO12)
- net ~{LOCK}: now also U3.20 (DIO12); no longer U3.9 (DIO6)
- net ADC2: no longer names the net of U3.1 (ADC2)
- no-connect marks 8 -> 9
Other:
- company: (none) -> antoine163
- title: (none) -> Ble Smart Lock
- moved on the sheet: C9

Commit message: Mise a jour pcb en v1.1 et readme
Connections:
- net OPENED: now also U3.20 (DIO12); no longer U3.9 (DIO6)
- net ~{LOCK}: now also U3.9 (DIO6); no longer U3.20 (DIO12)
Changed lines of the file:
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@@
 	(title_block
 		(title "Ble Smart Lock")
-		(date "2024-03-30")
-		(rev "v1.0")
+		(date "2024-05-18")
+		(rev "v1.1")
 		(company "antoine163")
 	)
@@
 	(hierarchical_label "~{LOCK}"
 		(shape output)
-		(at 161.29 101.6 0)
+		(at 161.29 86.36 0)
 		(fields_autoplaced yes)
 		(effects
@@
 	(hierarchical_label "OPENED"
 		(shape input)
-		(at 161.29 86.36 0)
-		(fields_autoplaced yes)
-		(effects
+		(at 161.29 101.6 0)
+		(fields_autoplaced yes)
+		(effects
